File: Sloppy_Holley_Flex-over-can/Flex-over-can/Flex-over-can.kicad_sch (KiCad schematic)
At the start: 1 part, among them U1 ESP32-C3-SuperMini

Commit message: Add V001 schematic with Power and Connector sheets
- Root sheet: ESP32-C3-MINI-1, ME6211 3V3, TPS7B6950 sensor 5V,
  TJA1051T/3 CAN, USB-C, flex input, ADS1115 analog, 4x BTS3256D outputs.
- Power sheet: placeholder for own protection + 5V circuit
  (VBAT_IN/GND in, VBAT/+5V out).
- Connector sheet: 24 harness pin stubs ending in no-connect flags.
- Vendor Espressif KiCad lib 3.2.1 and custom FlexCAN symbols.
- Docs: sheet table, LCSC part list, progress log.

Co-Authored-By: Claude Opus 5.5 <noreply@anthropic.com>
Parts:
- removed U1: ESP32-C3-SuperMini, ESP32C3-SuperMini:ESP32-C3-SuperMini, symbol ESP32-C3-SuperMini:ESP32-C3-SuperMini
- added C10, C12, C13, C20, C21, C22, C23, C24, C30, C31, C32, C33: 100nF, Capacitor_SMD:C_0603_1608Metric, symbol Device:C
- added C11, C7: 1uF, Capacitor_SMD:C_0603_1608Metric, symbol Device:C
- added C14: 1nF, Capacitor_SMD:C_0603_1608Metric, symbol Device:C
- added C5: 1uF 50V, Capacitor_SMD:C_0805_2012Metric, symbol Device:C
- added C6: 2.2uF 50V, Capacitor_SMD:C_0805_2012Metric, symbol Device:C
- added C8, C9: 10uF, Capacitor_SMD:C_0603_1608Metric, symbol Device:C
- added D10, D11, D12, D13, D7: BAT54S, Package_TO_SOT_SMD:SOT-23, symbol Diode:BAT54S
- added D4: B5819W, Diode_SMD:D_SOD-123, symbol Device:D_Schottky
- added D5: STATUS, LED_SMD:LED_0603_1608Metric, symbol Device:LED
- added D6: NUP2105L, Package_TO_SOT_SMD:SOT-23, symbol Power_Protection:NUP2105L
- added F2: 0.2A 30V, Fuse:Fuse_1206_3216Metric, symbol Device:Polyfuse
- added J2: USB-C, Connector_USB:USB_C_Receptacle_HRO_TYPE-C-31-M-12, symbol Connector:USB_C_Receptacle_USB2.0_16P
- added JP1: CAN_TERM, Jumper:SolderJumper-2_P1.3mm_Open_RoundedPad1.0x1.5mm, symbol Jumper:SolderJumper_2_Open
- added NT1: NetTie_2, NetTie:NetTie-2_SMD_Pad0.5mm, symbol Device:NetTie_2
- added R10, R15, R4, R5, R6: 10k, Resistor_SMD:R_0603_1608Metric, symbol Device:R
- added R11: 120, Resistor_SMD:R_0603_1608Metric, symbol Device:R
- added R12, R13: 5.1k, Resistor_SMD:R_0603_1608Metric, symbol Device:R
- added R14, R8, R9: 4.7k, Resistor_SMD:R_0603_1608Metric, symbol Device:R
- added R20, R21, R22, R23: 12k, Resistor_SMD:R_0603_1608Metric, symbol Device:R
- added R24, R25, R26, R27: 20k, Resistor_SMD:R_0603_1608Metric, symbol Device:R
- added R30, R31, R32, R33: 3.3k, Resistor_SMD:R_0603_1608Metric, symbol Device:R
- added R34, R35, R36, R37: 100k, Resistor_SMD:R_0603_1608Metric, symbol Device:R
- added R38, R39, R40, R41: 15k DNP, Resistor_SMD:R_0603_1608Metric, symbol Device:R
- added R7: 1k, Resistor_SMD:R_0603_1608Metric, symbol Device:R
- added SW1: BOOT, Button_Switch_SMD:SW_Push_1P1T_XKB_TS-1187A, symbol Switch:SW_Push
- added U1: ESP32-C3-MINI-1-N4, Espressif:ESP32-C3-MINI-1, symbol Espressif:ESP32-C3-MINI-1
- added U10: ADS1115IDGSR, Package_SO:TSSOP-10_3x3mm_P0.5mm, symbol Analog_ADC:ADS1115IDGS
- added U11: ME6211C33M5G-N, Package_TO_SOT_SMD:SOT-23-5, symbol Regulator_Linear:AP2112K-3.3
- added U3: TPS7B6950QDCYRQ1, Package_TO_SOT_SMD:SOT-223, symbol FlexCAN:TPS7B6950QDCY
- added U4, U5, U6, U7: BTS3256D, Package_TO_SOT_SMD:TO-252-5_TabPin6, symbol FlexCAN:BTS3256D
- added U8: TJA1051T/3, Package_SO:SOIC-8_3.9x4.9mm_P1.27mm, symbol Interface_CAN_LIN:TJA1051T-3
- added U9: USBLC6-2SC6, Package_TO_SOT_SMD:SOT-23-6, symbol Power_Protection:USBLC6-2SC6
Connections:
- new net +3V3: C10.1, C13.1, C24.1, C8.1, C9.1, D10.2 (K), D11.2 (K), D12.2 (K), D13.2 (K), D7.2 (K), R10.1, R4.1, R5.1, R6.1, R7.1, R8.1, R9.1, U1.3 (3V3), U10.8 (VDD), U11.5 (VOUT), U8.5 (VIO)
- new net +5V: C12.1, C7.1, D4.1 (K), R14.1, U11.1 (VIN), U11.3 (EN), U8.3 (VCC)
- new net +5V_SENS: C6.1, U3.3 (OUT)
- new net AIN1: C20.1, D10.3 (COM), R20.2, R24.1, U10.4 (AIN0)
- new net AIN1_IN: R20.1
- new net AIN2: C21.1, D11.3 (COM), R21.2, R25.1, U10.5 (AIN1)
- new net AIN2_IN: R21.1
- new net AIN3: C22.1, D12.3 (COM), R22.2, R26.1, U10.6 (AIN2)
- new net AIN3_IN: R22.1
- new net AIN4: C23.1, D13.3 (COM), R23.2, R27.1, U10.7 (AIN3)
- new net AIN4_IN: R23.1
- new net BOOT: R5.2, SW1.1, U1.23 (GPIO9)
- new net CANH: D6.1 (K), R11.1, U8.7 (CANH)
- new net CANL: D6.2 (K), JP1.2 (B), U8.6 (CANL)
- new net CAN_RX: U1.19 (GPIO5/ADC2_CH0), U8.4 (RXD)
- new net CAN_S: R10.2, U1.31 (GPIO21/U0TXD), U8.8 (S)
- new net CAN_TERM: JP1.1 (A), R11.2
- new net CAN_TX: U1.18 (GPIO4/ADC1_CH4), U8.1 (TXD)
- new net CC1: J2.A5 (CC1), R12.1
- new net CC2: J2.B5 (CC2), R13.1
- new net EN: C11.1, R4.2, U1.8 (EN/CHIP_PU)
- new net FLEX_12V: F2.2
- new net FLEX_SIG: C14.1, D7.3 (COM), R15.2, U1.6 (GPIO3/ADC1_CH3)
- new net FLEX_SIG_IN: R14.2, R15.1
- new net GND: C10.2, C11.2, C12.2, C13.2, C14.2, C20.2, C21.2, C22.2, C23.2, C24.2, C30.2, C31.2, C32.2, C33.2, C5.2, C6.2, C7.2, C8.2, C9.2, D10.1 (A), D11.1 (A), D12.1 (A), D13.1 (A), D6.3 (A), D7.1 (A), J2.A1 (GND), J2.A12 (GND), J2.B1 (GND), J2.B12 (GND), J2.SH (SHIELD), NT1.2, R12.2, R13.2, R24.2, R25.2, R26.2, R27.2, R34.2, R35.2, R36.2, R37.2, R38.2, R39.2, R40.2, R41.2, SW1.2, U1.1 (GND), U1.11 (GND), U1.14 (GND), U1.2 (GND), U1.36 (GND), U1.37 (GND), U1.38 (GND), U1.39 (GND), U1.40 (GND), U1.41 (GND), U1.42 (GND), U1.43 (GND), U1.44 (GND), U1.45 (GND), U1.46 (GND), U1.47 (GND), U1.48 (GND), U1.49 (GND), U1.50 (GND), U1.51 (GND), U1.52 (GND), U1.53 (GND), U10.1 (ADDR), U10.3 (GND), U11.2 (GND), U3.2 (GND), U3.4 (GND), U4.5 (GND), U5.5 (GND), U6.5 (GND), U7.5 (GND), U8.2 (GND), U9.2 (GND)
- new net GND_SENS: NT1.1
- new net LED_A: D5.2 (A), R7.2
- new net OUT1: U4.3 (DRAIN), U4.6 (DRAIN)
- new net OUT1_CTL: R30.1, R34.1, U1.12 (GPIO0/ADC1_CH0/XTAL_32K_P)
- new net OUT1_IN: R30.2, U4.2 (IN)
- new net OUT1_SRP: R38.1, U4.4 (SRP)
- new net OUT2: U5.3 (DRAIN), U5.6 (DRAIN)
- new net OUT2_CTL: R31.1, R35.1, U1.13 (GPIO1/ADC1_CH1/XTAL_32K_N)
- new net OUT2_IN: R31.2, U5.2 (IN)
- new net OUT2_SRP: R39.1, U5.4 (SRP)
- new net OUT3: U6.3 (DRAIN), U6.6 (DRAIN)
- new net OUT3_CTL: R32.1, R36.1, U1.21 (GPIO7)
- new net OUT3_IN: R32.2, U6.2 (IN)
- new net OUT3_SRP: R40.1, U6.4 (SRP)
- new net OUT4: U7.3 (DRAIN), U7.6 (DRAIN)
- new net OUT4_CTL: R33.1, R37.1, U1.16 (GPIO10)
- new net OUT4_IN: R33.2, U7.2 (IN)
- new net OUT4_SRP: R41.1, U7.4 (SRP)
- new net SCL: R9.2, U1.20 (GPIO6), U10.10 (SCL)
- new net SDA: R8.2, U1.22 (GPIO8), U10.9 (SDA)
- new net STATUS_LED: D5.1 (K), R6.2, U1.5 (GPIO2/ADC1_CH2)
- new net USB_DM: J2.A7 (D-), J2.B7 (D-), U1.26 (GPIO18/USB_D-), U9.3 (I/O2), U9.4 (I/O2)
- new net USB_DP: J2.A6 (D+), J2.B6 (D+), U1.27 (GPIO19/USB_D+), U9.1 (I/O1), U9.6 (I/O1)
- new net VBAT: C30.1, C31.1, C32.1, C33.1, C5.1, F2.1, U3.1 (IN), U4.1 (VS), U5.1 (VS), U6.1 (VS), U7.1 (VS)
- new net VBUS: D4.2 (A), J2.A4 (VBUS), J2.A9 (VBUS), J2.B4 (VBUS), J2.B9 (VBUS), U9.5 (VBUS)
- no-connect marks 0 -> 4
Other:
- added sheet Connector (Connector.kicad_sch)
- added sheet Power (Power.kicad_sch)
- note added: "ANALOG 0-5V: 12k/20k divider (x0.625, firmware ANALOG_SCALE=1.6), 100nF, BAT54S clamp -> ADS1115 @0x48. GND_SENS joins GND only at NT1 (star point near ADC)."
- note added: "CAN: TJA1051T/3. S pulled high = silent until firmware drives GPIO21 low. JP1 bridges 120R termination (default open)."
- note added: "FLEX: open-collector signal, 4.7k pull-up to 5V, 10k + BAT54S clamp to 3V3 into GPIO3. Sensor 12V via F2 PTC."
- note added: "OUTPUTS: BTS3256D HITFET, 7.5A nom, 12kHz max PWM, internal 40V active clamp. 3.3k series (fault readback), 100k pulldown holds OFF in reset. SRP open = fast slew; fit R38-41 to slow edges. Load current returns via J1 pins 2+24."
- note added: "POWER: input protection + 5V regulator are on the Power sheet (VBAT_IN in; VBAT protected 12V and +5V out). This sheet: ME6211 LDO 5V -> 3V3, short-proof sensor 5V (U3, 150mA), USB VBUS diode-ORed into +5V (D4)."

Commit message: Split schematic into 10 US Letter sheets
Move root circuitry into named hierarchical sheets: Supplies, MCU,
USB, CAN, Flex, Analog and Outputs, alongside the existing Power and
Connector sheets. Root now holds only sheet blocks and a page index.
Cross-sheet nets use global labels. Netlist unchanged (74 parts,
69 nets); ERC unchanged. Update the HARDWARE.md sheet table.

Co-Authored-By: Claude Opus 5.5 <noreply@anthropic.com>
Parts:
- removed C10, C12, C13, C20, C21, C22, C23, C24, C30, C31, C32, C33: 100nF, Capacitor_SMD:C_0603_1608Metric, symbol Device:C
- removed C11, C7: 1uF, Capacitor_SMD:C_0603_1608Metric, symbol Device:C
- removed C14: 1nF, Capacitor_SMD:C_0603_1608Metric, symbol Device:C
- removed C5: 1uF 50V, Capacitor_SMD:C_0805_2012Metric, symbol Device:C
- removed C6: 2.2uF 50V, Capacitor_SMD:C_0805_2012Metric, symbol Device:C
- removed C8, C9: 10uF, Capacitor_SMD:C_0603_1608Metric, symbol Device:C
- removed D10, D11, D12, D13, D7: BAT54S, Package_TO_SOT_SMD:SOT-23, symbol Diode:BAT54S
- removed D4: B5819W, Diode_SMD:D_SOD-123, symbol Device:D_Schottky
- removed D5: STATUS, LED_SMD:LED_0603_1608Metric, symbol Device:LED
- removed D6: NUP2105L, Package_TO_SOT_SMD:SOT-23, symbol Power_Protection:NUP2105L
- removed F2: 0.2A 30V, Fuse:Fuse_1206_3216Metric, symbol Device:Polyfuse
- removed J2: USB-C, Connector_USB:USB_C_Receptacle_HRO_TYPE-C-31-M-12, symbol Connector:USB_C_Receptacle_USB2.0_16P
- removed JP1: CAN_TERM, Jumper:SolderJumper-2_P1.3mm_Open_RoundedPad1.0x1.5mm, symbol Jumper:SolderJumper_2_Open
- removed NT1: NetTie_2, NetTie:NetTie-2_SMD_Pad0.5mm, symbol Device:NetTie_2
- removed R10, R15, R4, R5, R6: 10k, Resistor_SMD:R_0603_1608Metric, symbol Device:R
- removed R11: 120, Resistor_SMD:R_0603_1608Metric, symbol Device:R
- removed R12, R13: 5.1k, Resistor_SMD:R_0603_1608Metric, symbol Device:R
- removed R14, R8, R9: 4.7k, Resistor_SMD:R_0603_1608Metric, symbol Device:R
- removed R20, R21, R22, R23: 12k, Resistor_SMD:R_0603_1608Metric, symbol Device:R
- removed R24, R25, R26, R27: 20k, Resistor_SMD:R_0603_1608Metric, symbol Device:R
- removed R30, R31, R32, R33: 3.3k, Resistor_SMD:R_0603_1608Metric, symbol Device:R
- removed R34, R35, R36, R37: 100k, Resistor_SMD:R_0603_1608Metric, symbol Device:R
- removed R38, R39, R40, R41: 15k DNP, Resistor_SMD:R_0603_1608Metric, symbol Device:R
- removed R7: 1k, Resistor_SMD:R_0603_1608Metric, symbol Device:R
- removed SW1: BOOT, Button_Switch_SMD:SW_Push_1P1T_XKB_TS-1187A, symbol Switch:SW_Push
- removed U1: ESP32-C3-MINI-1-N4, Espressif:ESP32-C3-MINI-1, symbol Espressif:ESP32-C3-MINI-1
- removed U10: ADS1115IDGSR, Package_SO:TSSOP-10_3x3mm_P0.5mm, symbol Analog_ADC:ADS1115IDGS
- removed U11: ME6211C33M5G-N, Package_TO_SOT_SMD:SOT-23-5, symbol Regulator_Linear:AP2112K-3.3
- removed U3: TPS7B6950QDCYRQ1, Package_TO_SOT_SMD:SOT-223, symbol FlexCAN:TPS7B6950QDCY
- removed U4, U5, U6, U7: BTS3256D, Package_TO_SOT_SMD:TO-252-5_TabPin6, symbol FlexCAN:BTS3256D
- removed U8: TJA1051T/3, Package_SO:SOIC-8_3.9x4.9mm_P1.27mm, symbol Interface_CAN_LIN:TJA1051T-3
- removed U9: USBLC6-2SC6, Package_TO_SOT_SMD:SOT-23-6, symbol Power_Protection:USBLC6-2SC6
Connections:
- no-connect marks 4 -> 0
Other:
- added sheet 3V3 and Sensor 5V (Supplies.kicad_sch)
- added sheet Analog Inputs (Analog.kicad_sch)
- added sheet CAN Bus (CAN.kicad_sch)
- added sheet Flex Sensor Input (Flex.kicad_sch)
- added sheet Low-Side Outputs (Outputs.kicad_sch)
- added sheet MCU ESP32-C3 (MCU.kicad_sch)
- added sheet USB-C (USB.kicad_sch)
- note added: "FLEX-OVER-CAN V001 - TOP LEVEL. Each block below is its own page (double-click to open). Signals between pages use global labels; same name = same net on every page."
- note added: "PAGE INDEX 1 Top level (this page) 2 Power - input protection + 5V regulator (VBAT_IN -> VBAT, +5V) 3 Connector - 24-pin harness connector stubs 4 3V3 and Sensor 5V - ME6211 LDO, TPS7B69 sensor 5V, USB VBUS OR-ing 5 MCU ESP32-C3 - module, reset/boot, status LED, I2C pull-ups 6 USB-C - connector, CC resistors, USB ESD 7 CAN Bus - TJA1051T/3 transceiver, termination jumper, ESD 8 Flex Sensor Input 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"
- note removed: "ANALOG 0-5V: 12k/20k divider (x0.625, firmware ANALOG_SCALE=1.6), 100nF, BAT54S clamp -> ADS1115 @0x48. GND_SENS joins GND only at NT1 (star point near ADC)."
- note removed: "CAN: TJA1051T/3. S pulled high = silent until firmware drives GPIO21 low. JP1 bridges 120R termination (default open)."
- note removed: "FLEX: open-collector signal, 4.7k pull-up to 5V, 10k + BAT54S clamp to 3V3 into GPIO3. Sensor 12V via F2 PTC."
- note removed: "OUTPUTS: BTS3256D HITFET, 7.5A nom, 12kHz max PWM, internal 40V active clamp. 3.3k series (fault readback), 100k pulldown holds OFF in reset. SRP open = fast slew; fit R38-41 to slow edges. Load current returns via J1 pins 2+24."
- note removed: "POWER: input protection + 5V regulator are on the Power sheet (VBAT_IN in; VBAT protected 12V and +5V out). This sheet: ME6211 LDO 5V -> 3V3, short-proof sensor 5V (U3, 150mA), USB VBUS diode-ORed into +5V (D4)."
