File: Sloppy_Holley_Flex-over-can/Flex-over-can/Connector.kicad_sch (KiCad schematic)
At the start: 0 parts

Commit message: Add files via upload
Parts:
- added J1: HCCPHPE24BKA90F, KiCad_Footprints:24pinConnectorFootprint, symbol 24pinConnectorSymbol:HCCPHPE24BKA90F
Connections:
- net +5V_SENS: now also J1.B2, J1.B5, J1.C2, J1.C5
- net AIN1_IN: now also J1.B3
- net AIN2_IN: now also J1.B6
- net AIN3_IN: now also J1.C3
- net AIN4_IN: now also J1.C6
- net CANH: now also J1.A2
- net CANL: now also J1.A3
- net FLEX_12V: now also J1.A4
- net FLEX_SIG_IN: now also J1.A5
- net GND: now also J1.A7, J1.B1
- net GND_SENS: now also J1.A6, J1.B4, J1.B7, J1.C4, J1.C7
- net OUT1: now also J1.A8
- net OUT2: now also J1.B8
- net OUT3: now also J1.C1
- net OUT4: now also J1.C8
- net VBAT_IN: now also J1.A1
- no-connect marks 24 -> 0
Other:
- note added: "+12V in"
- note added: "CAN HIGH"
- note added: "CAN LOW"
- note added: "FLEX GND"
- note added: "FLEX POWER"
- note added: "FLEX SIGNAL"
- note added: "Ground"
- note added: "RELAY GND OUT 1"
- note added: "RELAY GND OUT 2"
- note added: "RELAY GND OUT 3"
- note added: "RELAY GND OUT 4"
- note removed: "HARNESS CONNECTOR (24 pin) - placeholder. Each pin ends in a no-connect flag. Place your connector, delete the X, wire its pin to the stub. GND pins 2 + 24 carry all output current. GND_SENS = quiet sensor ground (star-tied on main sheet, NT1)."
- note removed: "Pin 1 +12V in"
- note removed: "Pin 10 Output 3 (low side)"
- note removed: "Pin 11 Output 4 (low side)"
- note removed: "Pin 12 +5V sensor"
- note removed: "Pin 13 Analog 1 signal"
- note removed: "Pin 14 Sensor GND"
- note removed: "Pin 15 +5V sensor"
- note removed: "Pin 16 Analog 2 signal"
- note removed: "Pin 17 Sensor GND"
- note removed: "Pin 18 +5V sensor"
- note removed: "Pin 19 Analog 3 signal"
- note removed: "Pin 2 Power GND"
- note removed: "Pin 20 Sensor GND"
- note removed: "Pin 21 +5V sensor"
- note removed: "Pin 22 Analog 4 signal"
- note removed: "Pin 23 Sensor GND"
- note removed: "Pin 24 Power GND"
- note removed: "Pin 3 CAN H"
- note removed: "Pin 4 CAN L"
- note removed: "Pin 5 Flex sensor +12V out"
- note removed: "Pin 6 Flex sensor signal"
- note removed: "Pin 7 Flex sensor GND"
- note removed: "Pin 8 Output 1 (low side)"
- note removed: "Pin 9 Output 2 (low side)"
