File: Sloppy_Holley_Flex-over-can/Flex-over-can/Power.kicad_sch (KiCad schematic)
At the start: 0 parts

Commit message: Add files via upload
Parts:
- added C1: 10uF, Capacitor_SMD:C_0805_2012Metric, symbol Device:C_Polarized_US
- added C2, C3: 0.1uF, Capacitor_SMD:C_0805_2012Metric, symbol Device:C
- added C4: 47uF, Capacitor_Tantalum_SMD:CP_EIA-3528-21_Kemet-B, symbol Device:C_Polarized_US
- added D1: B130-13-F, Diode_SMD:D_SMA, symbol Device:D_Schottky
- added D2: 1SMB5919BT3G, Diode_SMD:D_SMB, symbol Device:D_Zener
- added RV1: Varistor, Diode_SMD:D_SMC, symbol Device:Varistor_US
- added U2: L7805ABD2T-TR, Package_TO_SOT_SMD:TO-263-2, symbol Regulator_Linear:L7805
Connections:
- net +5V: now also C3.1, C4.1, D2.1 (K), U2.3 (OUT)
- net GND: now also C1.2, C2.2, C3.2, C4.2, D2.2 (A), RV1.2, U2.2 (GND)
- net VBAT: now also D1.1 (K), U2.1 (IN)
- net VBAT_IN: now also C1.1, C2.1, D1.2 (A), RV1.1
Other:
- note added: "VOLTAGE REGULATOR"
- note removed: "POWER SUPPLY - placeholder for your input protection + 5V circuit. IN: VBAT_IN = raw +12V from connector pin 1. GND = power ground (pins 2 + 24). OUT: VBAT = protected +12V. Feeds sensor 5V reg U3 (150 mA max), flex PTC F2, BTS3256D VS pins. Budget ~250 mA. Output load current does not flow through VBAT. OUT: +5V = board 5V. ME6211 3V3 LDO (ESP32 WiFi peaks ~350 mA) + TJA1051 (~70 mA). Size for 0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"
