File: Sloppy_Holley_Flex-over-can/Flex-over-can/MCU.kicad_sch (KiCad schematic)
At the start: 12 parts, among them SW1 BOOT, U1 ESP32-C3-MINI-1-N4

Commit message: Review power/connector sheets, fix ERC, add 3D models for all parts
- Remove duplicate PWR_FLAG on +5V (ERC pin_to_pin error)
- Register KiCad_Footprints and 24pinConnectorSymbol libs for J1
- Correct D1 value to B160-13-F and RV1 to SMDJ24CA to match LCSC parts
- C1: 10uF 50V X5R 1206 (C13585) for load-dump margin
- F2: 0.2A/60V resettable PTC, Brightking SMD1812B020TF-J (C269125)
- Add STEP models for J1, J2 (USB-C), SW1 (BOOT) and fix ESP32 model path
- Project-local footprint copies carry the models for J2, SW1, F2

Co-Authored-By: Claude Opus 5.5 <noreply@anthropic.com>
Parts:
- SW1: footprint Button_Switch_SMD:SW_Push_1P1T_XKB_TS-1187A -> KiCad_Footprints:SW_Push_1P1T_XKB_TS-1187A
Changed lines of the file:
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@@
 			)
 		)
-		(property "Footprint" "Button_Switch_SMD:SW_Push_1P1T_XKB_TS-1187A"
+		(property "Footprint" "KiCad_Footprints:SW_Push_1P1T_XKB_TS-1187A"
 			(at 185.42 111.76 0)
 			(hide yes)

Commit message: Add PCB placement notes for decoupling caps to each sheet
Co-Authored-By: Claude Opus 5.5 <noreply@anthropic.com>
Other:
- note added: "PCB PLACEMENT NOTES: - C10 (100nF) at U1 pin 3 (3V3), smallest loop to GND pad. - C9 (10uF) next to C10, same 3V3 pin. - C11 (1uF) at U1 pin 8 (EN). - Keep-out: no copper or parts under/near U1 antenna end."
Changed lines of the file:
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@@
 		)
 	)
+  (text "PCB PLACEMENT NOTES:\n- C10 (100nF) at U1 pin 3 (3V3), smallest loop to GND pad.\n- C9 (10uF) next to C10, same 3V3 pin.\n- C11 (1uF) at U1 pin 8 (EN).\n- Keep-out: no copper or parts under/near U1 antenna end."
+    (at 15.24 180.34 0)
+    (effects (font (size 1.27 1.27) (color 0 0 194 1)) (justify left bottom))
+  )
 	(symbol
 		(lib_id "Device:R")
