File: Sloppy_Holley_Flex-over-can/Flex-over-can/Outputs.kicad_sch (KiCad schematic)
At the start: 20 parts, among them U4 BTS3256D, U5 BTS3256D, U6 BTS3256D, U7 BTS3256D

Commit message: Mark R38-R41 (SRP slew resistors) Do-not-populate
R38-R41 only had a "DNP" text field, so BOM and CPL exports would have
placed them. Set the real DNP attribute in the schematic and synced it
to the PCB. KiCad's save also normalized the sheets to LF line endings
and reformatted text notes; no other design changes.

Co-Authored-By: Claude Opus 5.5 <noreply@anthropic.com>
Parts:
- R38, R39, R40, R41: now not fitted
Changed lines of the file:
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@@
 	(generator_version "10.0")
 	(paper "USLetter")
+	(text "PCB PLACEMENT NOTES:\n- C30 at U4, C31 at U5, C32 at U6, C33 at U7 VBAT pin 1 (100nF each).\n- Wide copper on OUT tabs and the GND return to J1 A7/B1 (relay current)."
+		(exclude_from_sim no)
+		(at 15.24 180.34 0)
+		(effects
+			(font
+				(size 1.27 1.27)
+				(color 0 0 194 1)
+			)
+			(justify left bottom)
+		)
+	)
+	(text "OUTPUTS (x4): BTS3256D HITFET low-side, 7.5A nom, 12kHz max PWM, internal 40V active clamp.\n3.3k series (fault readback), 100k pulldown holds OFF in reset. SRP open = fast slew; fit R38-41 to slow edges.\nLoad current returns via J1 pins A7 + B1 (GND)."
+		(exclude_from_sim no)
+		(at 25.4 30.48 0)
+		(effects
+			(font
+				(size 2 2)
+				(bold yes)
+			)
+			(justify left bottom)
+		)
+	)
 	(wire
 		(pts
@@
 		)
 	)
-  (text "PCB PLACEMENT NOTES:\n- C30 at U4, C31 at U5, C32 at U6, C33 at U7 VBAT pin 1 (100nF each).\n- Wide copper on OUT tabs and the GND return to J1 A7/B1 (relay current)."
-    (at 15.24 180.34 0)
-    (effects (font (size 1.27 1.27) (color 0 0 194 1)) (justify left bottom))
-  )
-  (text "OUTPUTS (x4): BTS3256D HITFET low-side, 7.5A nom, 12kHz max PWM, internal 40V active clamp.\n3.3k series (fault readback), 100k pulldown holds OFF in reset. SRP open = fast slew; fit R38-41 to slow edges.\nLoad current returns via J1 pins A7 + B1 (GND)."
-    (at 25.4 30.48 0)
-    (effects (font (size 2 2) (bold yes)) (justify left bottom))
-  )
 	(symbol
 		(lib_id "Device:R")
@@
 		(on_board yes)
 		(in_pos_files yes)
-		(dnp no)
+		(dnp yes)
 		(property "Reference" "R38"
 			(at 57.912 96.52 90)
@@
 		(on_board yes)
 		(in_pos_files yes)
-		(dnp no)
+		(dnp yes)
 		(property "Reference" "R40"
 			(at 57.912 157.48 90)
@@
 		(on_board yes)
 		(in_pos_files yes)
-		(dnp no)
+		(dnp yes)
 		(property "Reference" "R39"
 			(at 179.832 96.52 90)
@@
 		(on_board yes)
 		(in_pos_files yes)
-		(dnp no)
+		(dnp yes)
 		(property "Reference" "R41"
 			(at 179.832 157.48 90)
